File: kicad/eth68/eth68.kicad_sch (KiCad schematic)
At the start: 70 parts, among them J1 Conn_01x03_Pin, J14 Conn_02x10_Odd_Even, J201 Conn_01x02_Pin, J3 Conn_01x02_Pin, U201 PCM3168APAPR, U5 STM32H743ZIT6, Y1 SG-210STF

Commit message: WIP
Connections:
- net GPIO3 renamed OSC_RESET
Other:
- note added: "TIM16_CH1 previously, now using as UART7"
- note added: "TODO- * wire i2c to pcm3168 * wire up gpio to reset lines of codec and phy * look at next-rev notes for proto boards * pull downs on analog outputs, far side of caps * thermal pad vias for PCM3168 * add GPIO * wire up USB lines * redo top/bottom gnd vias * jumpers for selecting modes, address, etc * check pin config in stm32cube"
- note removed: "TIM16_CH1 previously, now using UART7"
- note removed: "TODO- * wire i2c to pcm3168 * try re-pinning UART to pins 9-15 or 19-22 * GPIO for stopping audio clock * look at next-rev notes for proto boards * pull downs on analog outputs, far side of caps * thermal pad vias for PCM3168 * add GPIO * power switch * wire up USB lines * redo top/bottom gnd vias * jumpers for selecting modes, address, etc"
- moved on the sheet: H1, H2, H3, H4, H5, H6, H7

Commit message: WIP
Parts:
- removed J1: Conn_01x03_Pin, Connector_PinHeader_2.54mm:PinHeader_1x03_P2.54mm_Vertical, symbol Connector:Conn_01x03_Pin
- added R27, R29: 4.7k, Resistor_SMD:R_0603_1608Metric, symbol Device:R_Small
- added R63, R64, R65, R66: 0, Resistor_SMD:R_0603_1608Metric, symbol Device:R_Small
Connections:
- net VDD: now also R27.1, R29.1
- net at R202.1, U201.43 (MDI_SDA_DEMP): now also R64.1
- net CODEC_RESET: now reaches J201.2 (Pin_2), R208.2, U201.4 (RST_N)
- net CODEC_RESET: now also R65.2
- net at R201.2, U201.42 (MC_SCL_FMT): now also R63.1
- net at U5.12 (PF2): now also R65.1
- net I2C1_SCL: now reaches U5.136 (PB6)
- net I2C1_SCL: now also R27.2, R63.2
- net I2C1_SDA: now reaches U5.137 (PB7)
- net I2C1_SDA: now also R29.2, R64.2
- net at U5.14 (PF4): now also R66.1
- new net PHY_RESET: R66.2
Other:
- added sheet rs232 (rs232.kicad_sch)
- note added: "TODO- * wire up gpio to reset lines of codec and phy * look at next-rev notes for proto boards * pull downs on analog outputs, far side of caps * thermal pad vias for PCM3168 * add GPIO * wire up USB lines * redo top/bottom gnd vias * jumpers for selecting modes, address, etc * check pin config in stm32cube"
- note removed: "TODO- * wire i2c to pcm3168 * wire up gpio to reset lines of codec and phy * look at next-rev notes for proto boards * pull downs on analog outputs, far side of caps * thermal pad vias for PCM3168 * add GPIO * wire up USB lines * redo top/bottom gnd vias * jumpers for selecting modes, address, etc * check pin config in stm32cube"

Commit message: WIP
Other:
- note added: "TODO- * look at next-rev notes for proto boards * pull downs on analog outputs, far side of caps * thermal pad vias for PCM3168 * add GPIO * wire up USB lines * redo top/bottom gnd vias * jumpers for selecting modes, address, etc * check pin config in stm32cube"
- note removed: "TODO- * wire up gpio to reset lines of codec and phy * look at next-rev notes for proto boards * pull downs on analog outputs, far side of caps * thermal pad vias for PCM3168 * add GPIO * wire up USB lines * redo top/bottom gnd vias * jumpers for selecting modes, address, etc * check pin config in stm32cube"
Changed lines of the file:
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@@
 	(generator_version "9.0")
 	(paper "A1")
-	(text "TODO-\n* wire up gpio to reset lines of codec and phy\n* look at next-rev notes for proto boards\n* pull downs on analog outputs, far side of caps\n* thermal pad vias for PCM3168\n* add GPIO\n* wire up USB lines\n* redo top/bottom gnd vias\n* jumpers for selecting modes, address, etc\n* check pin config in stm32cube"
+	(text "TODO-\n* look at next-rev notes for proto boards\n* pull downs on analog outputs, far side of caps\n* thermal pad vias for PCM3168\n* add GPIO\n* wire up USB lines\n* redo top/bottom gnd vias\n* jumpers for selecting modes, address, etc\n* check pin config in stm32cube"
 		(exclude_from_sim no)
 		(at 853.694 477.266 0)
